File: k2_1.sch (KiCad schematic (older format))
At the start: 22 parts, among them IC1 TL074, J1 PJ301_THONKICONN6, J13 Conn_01x05_Female, J16 Conn_01x05_Male, J2 PJ301_THONKICONN6, J3 PJ301_THONKICONN6, J4 PJ301_THONKICONN6

Commit message: printing pretty schem
Changed lines of the file:
@@
 AR Path="/62AEB81D" Ref="D5"  Part="1"
 AR Path="/61896CD9/62AEB81D" Ref="D5"  Part="1"
-F 0 "D5" H 5700 3819 59  0000 L BNN
-F 1 "1N4148" H 5700 3709 59  0000 L BNN
+F 0 "D5" H 5550 3650 59  0000 L BNN
+F 1 "1N4148" H 5500 3550 59  0000 L BNN
 F 2 "Diode_SMD:D_1206_3216Metric_Pad1.42x1.75mm_HandSolder" H 5600 3800 50  0001 C CNN
 F 3 "" H 5600 3800 50  0001 C CNN
