File: k2_4.sch (KiCad schematic (older format))
At the start: 14 parts, among them IC1 TL074, IC2 TL072, IC3 TL074

Commit message: printing pretty schem
Other:
- note added: "Kinks had ferrite inductors on the input\ni've removed them\nmight want a 10R for noise suprpesison though???\nHad been S1JL but I like THT 1N5819"
- note added: "modified by karl.stamm@gmail.com\nfrom Kinks v4.1 to Crimps v1.x\nkarltron.com/crimps\n"
- note added: "reminder to later\nplay with these cap values\ni dont think they need to be so large\nseems to work sans a second set of 22u"
- note removed: "C9:"
- note removed: "Kinks had ferrite inductors on the input\ni've removed them\nmight want a 10R for noise suprpesison though???"
- note removed: "ceramic or tantalum"
- note removed: "eg AVX F981C475MMA"
- note removed: "modified by karl.stamm@gmail.com\nfrom Kinks v4.1 to Crimps v1.0.1\nkarltron.com/crimps\n"
- note removed: "reminder to later\nplay with these cap values\ni dont think they need to be so large"
Changed lines of the file:
@@
 Text Notes 9700 6950 0    85   ~ 0
 Power entry
-Text Notes 9100 2500 0    42   ~ 0
-eg AVX F981C475MMA
-Text Notes 9100 2400 0    42   ~ 0
-ceramic or tantalum
-Text Notes 9100 2300 0    42   ~ 0
-C9:
 Text Notes 7500 7150 0    85   ~ 0
 Émilie Gillet
@@
 	3050 3350 3100 3350
 Text Notes 6250 1600 0    50   ~ 0
-reminder to later\nplay with these cap values\ni dont think they need to be so large
+reminder to later\nplay with these cap values\ni dont think they need to be so large\nseems to work sans a second set of 22u
 Text Notes 2450 2500 0    50   ~ 0
-Kinks had ferrite inductors on the input\ni've removed them\nmight want a 10R for noise suprpesison though???
+Kinks had ferrite inductors on the input\ni've removed them\nmight want a 10R for noise suprpesison though???\nHad been S1JL but I like THT 1N5819
 Text Notes 7400 6450 0    50   ~ 0
-modified by karl.stamm@gmail.com\nfrom Kinks v4.1 to Crimps v1.0.1\nkarltron.com/crimps\n
+modified by karl.stamm@gmail.com\nfrom Kinks v4.1 to Crimps v1.x\nkarltron.com/crimps\n
 Wire Wire Line
 	3700 3350 3100 3350
